File: QCK.kicad_sch (KiCad schematic)
At the start: 208 parts, among them J1 Conn_01x05_Female, J2 USB_C_Receptacle_USB2.0, J3 Conn_01x03_Female, SW1 RotaryEncoder_Switch, SW2 SW_Push, SW3 SW_Push, U1 AMS1117-3.3, U2 STM32F072R8Tx, U3 SSD1306_128X64

Commit message: Routing Adjustment, Pinout Change for I2Cs and also SWDIO & SWCLK
Connections:
- net D_N: now also U2.44 (PA11); no longer U2.43 (PA10)
- net D_P: now also U2.45 (PA12); no longer U2.44 (PA11)
- net I2C_CLK: now also U2.61 (PB8); no longer U2.58 (PB6)
- net I2C_DAT: now also U2.62 (PB9); no longer U2.59 (PB7)
- net SWCLK: now also U2.49 (PA14); no longer U2.61 (PB8)
- net SWDIO: now also U2.46 (PA13); no longer U2.62 (PB9)
- net row5: now also U2.50 (PA15); no longer U2.49 (PA14)
- net PA9: no longer names the net of U2.57 (PB5)
- net PA9: no longer J3.1 (Pin_1)
- new net PB6: J3.1 (Pin_1), U2.58 (PB6)
Changed lines of the file:
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@@
   (junction (at 71.12 186.69) (diameter 0) (color 0 0 0 0)
   )
-  (no_connect (at 567.69 163.83))
   (no_connect (at 532.13 212.09))
-  (no_connect (at 567.69 171.45))
   (no_connect (at 532.13 207.01))
   (no_connect (at 567.69 186.69))
@@
   (no_connect (at 567.69 143.51))
   (no_connect (at 532.13 171.45))
+  (no_connect (at 567.69 194.31))
   (no_connect (at 544.83 101.6))
   (no_connect (at 532.13 209.55))
+  (no_connect (at 567.69 158.75))
   (no_connect (at 532.13 166.37))
   (no_connect (at 567.69 184.15))
@@
   (no_connect (at 532.13 214.63))
   (no_connect (at 532.13 163.83))
-  (no_connect (at 567.69 166.37))
+  (no_connect (at 567.69 189.23))
   (no_connect (at 544.83 104.14))
   (no_connect (at 567.69 146.05))
   (no_connect (at 532.13 204.47))
-  (wire (pts (xy 567.69 161.29) (xy 575.31 161.29))
-    (stroke (width 0) (type default) (color 0 0 0 0))
-  )
   (wire (pts (xy 547.37 128.27) (xy 549.91 128.27))
     (stroke (width 0) (type default) (color 0 0 0 0))
@@
     (stroke (width 0) (type default) (color 0 0 0 0))
   )
+  (wire (pts (xy 567.69 199.39) (xy 575.31 199.39))
+    (stroke (width 0) (type default) (color 0 0 0 0))
+  )
   (polyline (pts (xy 240.03 167.64) (xy 240.03 187.96))
     (stroke (width 0) (type default) (color 0 0 0 0))
@@
     (stroke (width 0) (type default) (color 0 0 0 0))
   )
+  (wire (pts (xy 567.69 166.37) (xy 575.31 166.37))
+    (stroke (width 0) (type default) (color 0 0 0 0))
+  )
   (wire (pts (xy 350.52 161.29) (xy 360.68 161.29))
     (stroke (width 0) (type default) (color 0 0 0 0))
@@
     (stroke (width 0) (type default) (color 0 0 0 0))
   )
-  (wire (pts (xy 567.69 189.23) (xy 575.31 189.23))
-    (stroke (width 0) (type default) (color 0 0 0 0))
-  )
   (wire (pts (xy 172.72 204.47) (xy 160.02 204.47))
     (stroke (width 0) (type default) (color 0 0 0 0))
@@
     (stroke (width 0) (type default) (color 0 0 0 0))
   )
-  (wire (pts (xy 567.69 191.77) (xy 575.31 191.77))
-    (stroke (width 0) (type default) (color 0 0 0 0))
-  )
   (polyline (pts (xy 170.18 119.38) (xy 170.18 139.7))
     (stroke (width 0) (type default) (color 0 0 0 0))
@@
     (stroke (width 0) (type default) (color 0 0 0 0))
   )
-  (wire (pts (xy 567.69 196.85) (xy 575.31 196.85))
-    (stroke (width 0) (type default) (color 0 0 0 0))
-  )
   (polyline (pts (xy 394.97 139.7) (xy 394.97 119.38))
     (stroke (width 0) (type default) (color 0 0 0 0))
@@
     (stroke (width 0) (type default) (color 0 0 0 0))
   )
+  (wire (pts (xy 567.69 163.83) (xy 575.31 163.83))
+    (stroke (width 0) (type default) (color 0 0 0 0))
+  )
   (wire (pts (xy 147.32 165.1) (xy 168.91 165.1))
     (stroke (width 0) (type default) (color 0 0 0 0))
@@
     (stroke (width 0) (type default) (color 0 0 0 0))
   )
-  (wire (pts (xy 567.69 158.75) (xy 575.31 158.75))
-    (stroke (width 0) (type default) (color 0 0 0 0))
-  )
   (polyline (pts (xy 45.72 252.73) (xy 66.04 252.73))
     (stroke (width 0) (type default) (color 0 0 0 0))
@@
     (stroke (width 0) (type default) (color 0 0 0 0))
   )
-  (wire (pts (xy 567.69 168.91) (xy 575.31 168.91))
+  (polyline (pts (xy 181.61 209.55) (xy 201.93 209.55))
     (stroke (width 0) (type default) (color 0 0 0 0))
   )
-  (polyline (pts (xy 181.61 209.55) (xy 201.93 209.55))
+  (wire (pts (xy 567.69 171.45) (xy 575.31 171.45))
     (stroke (width 0) (type default) (color 0 0 0 0))
   )
@@
     (stroke (width 0) (type default) (color 0 0 0 0))
   )
+  (wire (pts (xy 567.69 191.77) (xy 575.31 191.77))
+    (stroke (width 0) (type default) (color 0 0 0 0))
+  )
   (wire (pts (xy 570.23 38.1) (xy 570.23 41.91))
     (stroke (width 0) (type default) (color 0 0 0 0))
@@
     (stroke (width 0) (type default) (color 0 0 0 0))
   )
+  (wire (pts (xy 567.69 161.29) (xy 575.31 161.29))
+    (stroke (width 0) (type default) (color 0 0 0 0))
+  )
   (polyline (pts (xy 100.33 232.41) (xy 125.73 232.41))
     (stroke (width 0) (type default) (color 0 0 0 0))
@@
     (stroke (width 0) (type default) (color 0 0 0 0))
   )
+  (wire (pts (xy 567.69 196.85) (xy 575.31 196.85))
+    (stroke (width 0) (type default) (color 0 0 0 0))
+  )
   (polyline (pts (xy 127 252.73) (xy 152.4 252.73))
     (stroke (width 0) (type default) (color 0 0 0 0))
@@
     (stroke (width 0) (type default) (color 0 0 0 0))
   )
-  (wire (pts (xy 567.69 199.39) (xy 575.31 199.39))
-    (stroke (width 0) (type default) (color 0 0 0 0))
-  )
   (wire (pts (xy 116.84 199.39) (xy 113.03 199.39))
     (stroke (width 0) (type default) (color 0 0 0 0))
@@
     (stroke (width 0) (type default) (color 0 0 0 0))
   )
+  (wire (pts (xy 567.69 168.91) (xy 575.31 168.91))
+    (stroke (width 0) (type default) (color 0 0 0 0))
+  )
   (wire (pts (xy 375.92 229.87) (xy 402.59 229.87))
     (stroke (width 0) (type default) (color 0 0 0 0))
@@
     (stroke (width 0) (type default) (color 0 0 0 0))
   )
-  (wire (pts (xy 567.69 194.31) (xy 575.31 194.31))
-    (stroke (width 0) (type default) (color 0 0 0 0))
-  )
   (wire (pts (xy 354.33 204.47) (xy 354.33 226.06))
     (stroke (width 0) (type default) (color 0 0 0 0))
@@
     )
   )
-  (global_label "PA9" (shape input) (at 501.65 49.53 180) (fields_autoplaced)
+  (global_label "PB6" (shape input) (at 501.65 49.53 180) (fields_autoplaced)
     (effects (font (size 1.27 1.27)) (justify right))
-    (property "Intersheet References" "${INTERSHEET_REFS}" (id 0) (at 495.6688 49.6094 0)
+    (property "Intersheet References" "${INTERSHEET_REFS}" (id 0) (at 495.4874 49.4506 0)
       (effects (font (size 1.27 1.27)) (justify right) hide)
     )
@@
     )
   )
-  (global_label "row5" (shape input) (at 575.31 168.91 0) (fields_autoplaced)
+  (global_label "row5" (shape input) (at 575.31 171.45 0) (fields_autoplaced)
     (effects (font (size 1.27 1.27)) (justify left))
-    (property "Intersheet References" "${INTERSHEET_REFS}" (id 0) (at 582.1983 168.8306 0)
+    (property "Intersheet References" "${INTERSHEET_REFS}" (id 0) (at 582.1983 171.3706 0)
       (effects (font (size 1.27 1.27)) (justify left) hide)
     )
@@
     )
   )
-  (global_label "I2C_CLK" (shape input) (at 575.31 191.77 0) (fields_autoplaced)
+  (global_label "I2C_CLK" (shape input) (at 575.31 196.85 0) (fields_autoplaced)
     (effects (font (size 1.27 1.27)) (justify left))
-    (property "Intersheet References" "${INTERSHEET_REFS}" (id 0) (at 585.3431 191.6906 0)
+    (property "Intersheet References" "${INTERSHEET_REFS}" (id 0) (at 585.3431 196.7706 0)
       (effects (font (size 1.27 1.27)) (justify left) hide)
     )
@@
     )
   )
-  (global_label "D_N" (shape input) (at 575.31 158.75 0) (fields_autoplaced)
+  (global_label "D_N" (shape input) (at 575.31 161.29 0) (fields_autoplaced)
     (effects (font (size 1.27 1.27)) (justify left))
-    (property "Intersheet References" "${INTERSHEET_REFS}" (id 0) (at 581.2912 158.6706 0)
+    (property "Intersheet References" "${INTERSHEET_REFS}" (id 0) (at 581.2912 161.2106 0)
       (effects (font (size 1.27 1.27)) (justify left) hide)
     )
@@
     )
   )
-  (global_label "D_P" (shape input) (at 575.31 161.29 0) (fields_autoplaced)
+  (global_label "D_P" (shape input) (at 575.31 163.83 0) (fields_autoplaced)
     (effects (font (size 1.27 1.27)) (justify left))
-    (property "Intersheet References" "${INTERSHEET_REFS}" (id 0) (at 581.2307 161.2106 0)
+    (property "Intersheet References" "${INTERSHEET_REFS}" (id 0) (at 581.2307 163.7506 0)
       (effects (font (size 1.27 1.27)) (justify left) hide)
     )
@@
     )
   )
-  (global_label "PA9" (shape input) (at 575.31 189.23 0) (fields_autoplaced)
+  (global_label "PB6" (shape input) (at 575.31 191.77 0) (fields_autoplaced)
     (effects (font (size 1.27 1.27)) (justify left))
-    (property "Intersheet References" "${INTERSHEET_REFS}" (id 0) (at 581.2912 189.1506 0)
+    (property "Intersheet References" "${INTERSHEET_REFS}" (id 0) (at 581.4726 191.6906 0)
       (effects (font (size 1.27 1.27)) (justify left) hide)
     )
@@
     )
   )
-  (global_label "SWCLK" (shape input) (at 575.31 196.85 0) (fields_autoplaced)
+  (global_label "SWCLK" (shape input) (at 575.31 168.91 0) (fields_autoplaced)
     (effects (font (size 1.27 1.27)) (justify left))
-    (property "Intersheet References" "${INTERSHEET_REFS}" (id 0) (at 583.9521 196.7706 0)
+    (property "Intersheet References" "${INTERSHEET_REFS}" (id 0) (at 583.9521 168.8306 0)
       (effects (font (size 1.27 1.27)) (justify left) hide)
     )
@@
     )
   )
-  (global_label "SWDIO" (shape input) (at 575.31 199.39 0) (fields_autoplaced)
+  (global_label "SWDIO" (shape input) (at 575.31 166.37 0) (fields_autoplaced)
     (effects (font (size 1.27 1.27)) (justify left))
-    (property "Intersheet References" "${INTERSHEET_REFS}" (id 0) (at 583.5893 199.3106 0)
+    (property "Intersheet References" "${INTERSHEET_REFS}" (id 0) (at 583.5893 166.2906 0)
       (effects (font (size 1.27 1.27)) (justify left) hide)
     )
@@
     )
   )
-  (global_label "I2C_DAT" (shape input) (at 575.31 194.31 0) (fields_autoplaced)
+  (global_label "I2C_DAT" (shape input) (at 575.31 199.39 0) (fields_autoplaced)
     (effects (font (size 1.27 1.27)) (justify left))
-    (property "Intersheet References" "${INTERSHEET_REFS}" (id 0) (at 585.1012 194.2306 0)
+    (property "Intersheet References" "${INTERSHEET_REFS}" (id 0) (at 585.1012 199.3106 0)
       (effects (font (size 1.27 1.27)) (justify left) hide)
     )
